File: PCB/8Mux.kicad_sch (KiCad schematic)
At the start: 1 part, among them U27 74HC4051

Commit message: Updated PCB
Parts:
- removed U27: 74HC4051, symbol 74xx:74HC4051
- added U12: 74HC4051, Package_SO:TSSOP-16_4.4x5mm_P0.65mm, symbol 74xx:74HC4051
Connections:
- net GND: now also U12.7 (VEE), U12.8 (GND)
- net IN: now also U12.3 (A)
- net OUT0: now also U12.13 (A0)
- net OUT1: now also U12.14 (A1)
- net OUT2: now also U12.15 (A2)
- net OUT3: now also U12.12 (A3)
- net OUT4: now also U12.1 (A4)
- net OUT5: now also U12.5 (A5)
- net OUT6: now also U12.2 (A6)
- net OUT7: now also U12.4 (A7)
- net S0: now also U12.11 (S0)
- net S1: now also U12.10 (S1)
- net S2: now also U12.9 (S2)
- new net +3.3V: U12.16 (VCC)
- new net ~{EN}: U12.6 (~{E})
