File: PCB/CM5_GPIO.kicad_sch (KiCad schematic)
At the start: 26 parts, among them J1 RTC Connector, J14 JST_SHBM04B-SRSS-TB, J2 Conn_02x07_Odd_Even, J3 Conn_01x03, J7 Micro_SD_Card_Det, J8 THD-20-R, J9 THD-02-R, SW1 Right angle Tact button, U1 TPD4EUSB30, U18 RT9742GGJ5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

Commit message: Updated PCB
Parts:
- removed C5: 10u, Capacitor_SMD:C_0805_2012Metric, symbol Device:C
- removed J3: Conn_01x03, Connector_PinHeader_2.54mm:PinHeader_1x03_P2.54mm_Vertical, symbol Connector_Generic:Conn_01x03
- removed J7: Micro_SD_Card_Det, CM5IO:SDCARD_MOLEX_503398-1892, symbol Connector:Micro_SD_Card_Det2
- removed J8: THD-20-R, Connector_PinHeader_2.54mm:PinHeader_2x20_P2.54mm_Vertical, symbol Connector_Generic:Conn_02x20_Odd_Even
- removed R4: nf, Resistor_SMD:R_0805_2012Metric_Pad1.20x1.40mm_HandSolder, symbol Device:R
- removed R5: 0R, Resistor_SMD:R_0805_2012Metric_Pad1.20x1.40mm_HandSolder, symbol Device:R
- removed SW1: Right angle Tact button, Button_Switch_THT:SW_Tactile_SPST_Angled_PTS645Vx58-2LFS, symbol Switch:SW_Push
- removed TP3: TestPoint, TestPoint:TestPoint_Pad_2.0x2.0mm, symbol Connector:TestPoint
- removed U18: RT9742GGJ5, Package_TO_SOT_SMD:SOT-23-5, symbol CM5IO:RT9742GGJ5
- removed U5: 74LVC1G07SE-7, Package_TO_SOT_SMD:SOT-353_SC-70-5, symbol CM5IO:74LVC1G07_copy
- added J11: Raspberry_Pi_2_3, Connector_PinHeader_2.54mm:PinHeader_2x20_P2.54mm_Vertical, symbol Connector:Raspberry_Pi_2_3
- C1: value 100n -> 100nF; footprint Capacitor_SMD:C_0402_1005Metric -> Capacitor_SMD:C_0603_1608Metric_Pad1.08x0.95mm_HandSolder
- J14: renamed from J2; footprint Connector_PinHeader_2.54mm:PinHeader_2x07_P2.54mm_Vertical -> Connector_PinHeader_1.27mm:PinHeader_2x07_P1.27mm_Vertical
- R2: renamed from R1; value 1k -> 1kΩ; footprint Resistor_SMD:R_0402_1005Metric -> Resistor_SMD:R_0603_1608Metric_Pad0.98x0.95mm_HandSolder
- R3: renamed from R10; value 1k -> 50Ω; footprint Resistor_SMD:R_0402_1005Metric -> Resistor_SMD:R_0603_1608Metric_Pad0.98x0.95mm_HandSolder
- R4: renamed from R2; value 470R -> 470Ω; footprint Resistor_SMD:R_0402_1005Metric -> Resistor_SMD:R_0603_1608Metric_Pad0.98x0.95mm_HandSolder
- R5: renamed from R3; value 470R -> 470Ω; footprint Resistor_SMD:R_0402_1005Metric -> Resistor_SMD:R_0603_1608Metric_Pad0.98x0.95mm_HandSolder
- renumbered D2 to D1, D1 to D2, J14 to J12, J1 to J13, TP5 to TP2
Connections:
- net GPIO_VREF is gone; now on net +3.3V: Module1.78 (GPIO_VREF(1.8v/3.3v_Input))
- net GND: now also J11.14 (GND), J11.20 (GND), J11.25 (GND), J11.30 (GND), J11.34 (GND), J11.39 (GND), J11.6 (GND), J11.9 (GND)
- net GPIO12: now also J11.32 (PWM0/GPIO12)
- net GPIO13: now also J11.33 (PWM1/GPIO13)
- net GPIO14: now also J11.8 (GPIO14/TXD)
- net GPIO15: now also J11.10 (GPIO15/RXD)
- net GPIO16: now also J11.36 (GPIO16)
- net GPIO17: now also J11.11 (GPIO17)
- net GPIO18: now also J11.12 (GPIO18/PWM0)
- net GPIO19: now also J11.35 (GPIO19/MISO1)
- net GPIO20: now also J11.38 (GPIO20/MOSI1)
- net GPIO21: now also J11.40 (GPIO21/SCLK1)
- net GPIO22: now also J11.15 (GPIO22)
- net GPIO23: now also J11.16 (GPIO23)
- net GPIO24: now also J11.18 (GPIO24)
- net GPIO25: now also J11.22 (GPIO25)
- net GPIO26: now also J11.37 (GPIO26)
- net GPIO27: now also J11.13 (GPIO27)
- net GPIO4: now also J11.7 (GCLK0/GPIO4)
- net GPIO5: now also J11.29 (GCLK1/GPIO5)
- net GPIO6: now also J11.31 (GCLK2/GPIO6)
- net GPIO7: now also J11.26 (~{CE1}/GPIO7)
- net GPIO8: now also J11.24 (~{CE0}/GPIO8)
- net nPWR_LED: now also R3.2
- net +1.8v renamed +1V8
- net +3.3v renamed +3.3V
- net +3.3V: now also J11.1 (3V3), J11.17 (3V3)
- net +5v renamed +5V
- net +5V: now also J11.2 (5V), J11.4 (5V)
- net BT_nDis: no longer names the net of Module1.91 (BT_nDisable)
- net CC1: no longer names the net of Module1.94 (CC1)
- net CC2: no longer names the net of Module1.96 (CC2)
- net GPIO10 renamed MOSI0
- net MOSI0: now also J11.19 (MOSI0/GPIO10)
- net GPIO11 renamed CLK0
- net CLK0: now also J11.23 (SCLK0/GPIO11)
- net GPIO2 renamed GPIOSDA
- net GPIOSDA: now also J11.3 (SDA/GPIO2)
- net GPIO3 renamed GPIOSCL
- net GPIOSCL: now also J11.5 (SCL/GPIO3)
- net GPIO9 renamed MISO0
- net MISO0: now also J11.21 (MISO0/GPIO9)
- net ID_SC renamed ID_SCL
- net ID_SCL: now also J11.28 (ID_SC/GPIO1)
- net ID_SD renamed ID_SDA
- net ID_SDA: now also J11.27 (ID_SD/GPIO0)
- net WL_nDis: no longer names the net of Module1.89 (WiFi_nDisable)
- no-connect marks 9 -> 10
Other:
- note removed: "40Way GPIO Header"
- note removed: "CM5Lite SDCARD I/F"
- note removed: "GPIO Voltage select"
- note removed: "Not Fitted header"
- note removed: "PWR LED"
- moved on the sheet: D2, R3, TP2
