File: PCB/CM5_HighSpeed.kicad_sch (KiCad schematic)
At the start: 19 parts, among them J10 690-019-298-412, J12 USB3_A, J16 Conn_01x22_Female, J22 690-019-298-412, J5 Conn_01x22_Female, J6 THD-02-R, U12 RT9742SNGV, U6 AP22653W6

Commit message: Updated PCB
Parts:
- removed C12, C13: 100n, Capacitor_SMD:C_0402_1005Metric, symbol Device:C
- removed C2, C7, C8: 10u, Capacitor_SMD:C_0805_2012Metric, symbol Device:C
- removed C3: 100uF, Capacitor_Tantalum_SMD:CP_EIA-7343-31_Kemet-D, symbol Device:C_Polarized
- removed J12: USB3_A, CM5IO:MTCONN_UBAF30-D2011, symbol CM5IO:USB3_A
- removed J6: THD-02-R, Connector_PinHeader_2.54mm:PinHeader_2x02_P2.54mm_Vertical, symbol Connector_Generic:Conn_02x02_Odd_Even
- removed R12: 15K 1%, Resistor_SMD:R_0402_1005Metric, symbol Device:R
- removed R6, R7: 2.2K 1%, Resistor_SMD:R_0402_1005Metric, symbol Device:R
- removed U12: RT9742SNGV, Package_TO_SOT_SMD:TSOT-23_HandSoldering, symbol CM5IO:RT9742SNGV
- removed U6: AP22653W6, Package_TO_SOT_SMD:SOT-23-6, symbol CM5IO:AP2553W6
- added J4: USB3_A, Connector_USB:USB3_A_Molex_48393-001, symbol Connector:USB3_A
- J7: renamed from J16; now not fitted
- R1: renamed from R8; footprint Resistor_SMD:R_0402_1005Metric -> Resistor_SMD:R_0603_1608Metric_Pad0.98x0.95mm_HandSolder; now not fitted
- renumbered J22 to J6, J10 to J8
Connections:
- net GND: now also J4.10 (SHIELD), J4.4 (GND), J4.7 (DRAIN)
- net USB3-0-D_N: now also J4.2 (D-)
- net USB3-0-D_P: now also J4.3 (D+)
- net USB3-0-RX_N: now also J4.5 (SSRX-)
- net USB3-0-RX_P: now also J4.6 (SSRX+)
- net USB3-0-TX_N: now also J4.8 (SSTX-)
- net USB3-0-TX_P: now also J4.9 (SSTX+)
- net +3.3v renamed +3.3V
- net HDMI_5v renamed +5V
- net +5V: now also J4.1 (VBUS)
- net PCIE_PWR_EN: no longer names the net of Module1.106 (PCIE_PWR_EN)
- net SCL1 renamed ID_SCL
- net SDA1 renamed ID_SDA
- net USB3-1-D_N renamed USB3D_N
- net USB3-1-D_P renamed USB3D_P
- net USB3-1-RX_N renamed USB3RX_N
- net USB3-1-RX_P renamed USB3RX_P
- net USB3-1-TX_N renamed USB3TX_N
- net USB3-1-TX_P renamed USB3TX_P
- net VBUS_EN: no longer names the net of Module1.111 (VBUS_EN)
- no-connect marks 4 -> 5
Other:
- note removed: "Current Limit switch"
- note removed: "Jumpers to be fitted if DPHY1 is used"
