File: PCB/MM.kicad_sch (KiCad schematic)
At the start: 4 parts, among them Q1 2N7002, Q2 2N7002, U4 PINA780BIDEKR

Commit message: Updated PCB
Parts:
- added J16: Conn_01x02_Pin, Connector_PinHeader_1.27mm:PinHeader_1x02_P1.27mm_Vertical, symbol Connector:Conn_01x02_Pin
- R7: renamed from R11; footprint (none) -> Resistor_SMD:R_0603_1608Metric_Pad0.98x0.95mm_HandSolder
- renumbered U4 to U6
Connections:
- net GND: now also Q2.2 (S); no longer Q2.3 (D)
- net V+: now also J16.1 (Pin_1)
- net V-: now also Q2.3 (D); no longer Q2.2 (S)
- net at Q1.3 (D), R7.1: now also J16.2 (Pin_2)
Other:
- moved on the sheet: Q1, Q2
