File: PCB/Mux.kicad_sch (KiCad schematic)
At the start: 48 parts

Commit message: Updated PCB
Parts:
- removed TP12, TP13, TP14, TP15, TP16, TP17, TP18, TP19, TP28, TP29, TP30, TP31, TP32, TP33, TP34, TP35, TP44, TP45, TP46, TP47, TP48, TP49, TP50, TP51, TP60, TP61, TP62, TP63, TP64, TP65, TP66, TP67, TP76, TP77, TP78, TP79, TP80, TP81, TP82, TP83, TP92, TP93, TP94, TP95, TP96, TP97, TP98, TP99: TestPoint_Small, TestPoint:TestPoint_Pad_D1.0mm, symbol Connector:TestPoint_Small
- added J18: Conn_01x12_Pin, Connector_PinHeader_1.27mm:PinHeader_1x12_P1.27mm_Vertical, symbol Connector:Conn_01x12_Pin
Connections:
- net S0: now also J18.7 (Pin_7)
- net S1: now also J18.8 (Pin_8)
- net S2: now also J18.9 (Pin_9)
- new net +3.3V: J18.11 (Pin_11)
- new net 1:8 Mux9/OUT2: J18.1 (Pin_1)
- new net 1:8 Mux9/OUT3: J18.2 (Pin_2)
- new net 1:8 Mux9/OUT4: J18.3 (Pin_3)
- new net 1:8 Mux9/OUT5: J18.4 (Pin_4)
- new net 1:8 Mux9/OUT6: J18.5 (Pin_5)
- new net 1:8 Mux9/OUT7: J18.6 (Pin_6)
- new net GND: J18.12 (Pin_12)
- new net ~{EN}: J18.10 (Pin_10)
Other:
- removed sheet 1:8 Mux
- removed sheet 1:8 Mux3
- removed sheet 1:8 Mux4
- removed sheet 1:8 Mux5
- removed sheet 1:8 Mux6
- removed sheet 1:8 Mux7
- removed sheet 1:8 Mux8
- added sheet 1:8 Mux9 (8Mux.kicad_sch)
- sheet 1:8 Mux1 ports: added ~{EN}; removed EN
- sheet 1:8 Mux2 ports: added ~{EN}; removed EN
