File: PCB/PCIe-M2.kicad_sch (KiCad schematic)
At the start: 24 parts, among them J4 Bus_M.2_Socket_M, M1 M.2 Screw, M2 M.2 Solder Nut, M3 M.2 Solder Nut, M4 M.2 Solder Nut, M5 M.2 Solder Nut, U7 ASEK-32.768KHZ-L-R-T, U8 AP3441SHE-7B

Commit message: Updated PCB
Parts:
- removed C10, C19: 100n, Capacitor_SMD:C_0402_1005Metric, symbol Device:C
- removed C11: 4.7nF, Capacitor_SMD:C_0402_1005Metric, symbol Device:C
- removed C14, C15, C16, C17, C4, C6: 10u, Capacitor_SMD:C_0805_2012Metric, symbol Device:C
- removed L1: 2.2uH, CM5IO:L_Bourns_SRP5030CC, symbol Device:L
- removed R14: 100K 1%, Resistor_SMD:R_0402_1005Metric, symbol Device:R
- removed R15: 10K 1%, Resistor_SMD:R_0402_1005Metric, symbol Device:R
- removed R16: 2.2K 1%, Resistor_SMD:R_0402_1005Metric, symbol Device:R
- removed TP1: TestPoint, TestPoint:TestPoint_Pad_2.0x2.0mm, symbol Connector:TestPoint
- removed U7: ASEK-32.768KHZ-L-R-T, Crystal:Crystal_SMD_3225-4Pin_3.2x2.5mm, symbol CM5IO:ASEK-32.768KHZ-L-R-T
- removed U8: AP3441SHE-7B, Package_DFN_QFN:DFN-8-1EP_2x2mm_P0.5mm_EP1.05x1.75mm, symbol CM5IO:AP3441SHE-7B
- added C3: 100nF, Capacitor_SMD:C_0603_1608Metric_Pad1.08x0.95mm_HandSolder, symbol Device:C
- added X1: ASEK-32.768KHZ-L-R-T, Oscillator:Oscillator_SMD_Abracon_ASE-4Pin_3.2x2.5mm, symbol Oscillator:ASE-xxxMHz
- R6: renamed from R17; footprint Resistor_SMD:R_0402_1005Metric -> Resistor_SMD:R_0603_1608Metric_Pad0.98x0.95mm_HandSolder
- renumbered J4 to J15, M5 to M1, M4 to M2, M2 to M4, M1 to M5
Connections:
- net GND: now also C3.2, X1.2 (GND)
- net at J15.68 (SUSCLK): now also X1.3 (OUT)
- net M2_3v3 renamed +3.3V
- net +3.3V: now also C3.1, X1.1 (EN), X1.4 (Vdd)
- no-connect marks 15 -> 14
