File: PCB/PWR.kicad_sch (KiCad schematic)
At the start: 112 parts, among them J7 USB_C_Receptacle_USB2.0_16P, Q3 CSD17577Q3A, Q4 CSD17577Q3A, U10 BQ76905RGRR, U11 BQ25798RQMR, U14 TPS25730DREFR

Commit message: Updated PCB
Parts:
- removed C18, C19, C20, C22: 220nF, Capacitor_SMD:C_0402_1005Metric, symbol Device:C
- removed C19: 1nF, Capacitor_SMD:C_0402_1005Metric, symbol Device:C
- removed C21, C31, C32, C33, C34, C37, C38, C40, C41, C42, C45, C46: 10uF, Capacitor_SMD:C_0402_1005Metric, symbol Device:C
- removed C23, C25, C26, C27, C28, C30, C35, C36, C39, C48: .1uF, Capacitor_SMD:C_0402_1005Metric, symbol Device:C
- removed C24, C29: 100pF, Capacitor_SMD:C_0402_1005Metric, symbol Device:C
- removed C43, C47: 4.7uF, Capacitor_SMD:C_0402_1005Metric, symbol Device:C
- removed D3, D4, D5, D6, D7, D8: KT-0603R, LED_SMD:LED_0603_1608Metric, symbol Device:LED
- removed D7, D8: BZT52C39, Diode_SMD:D_SOD-123, symbol Device:D_Zener
- removed J7: USB_C_Receptacle_USB2.0_16P, Connector_USB:USB_C_Receptacle_G-Switch_GT-USB-7010ASV, symbol Connector:USB_C_Receptacle_USB2.0_16P
- removed Q3, Q4: CSD17577Q3A, Package_SON:VSON-8_3.3x3.3mm_P0.65mm_NexFET, symbol Transistor_FET:CSD17577Q3A
- removed R11, R26, R27, R28, R29, R30: 50Ω, Resistor_SMD:R_0402_1005Metric, symbol Device:R_US
- removed R12, R13, R18, R25: 100Ω, Resistor_SMD:R_0402_1005Metric, symbol Device:R_US
- removed R14: .001Ω, Resistor_SMD:R_0402_1005Metric, symbol Device:R_US
- removed R15, R16: 5.1kΩ, Resistor_SMD:R_0402_1005Metric, symbol Device:R_US
- removed R17: 10MΩ, Resistor_SMD:R_0402_1005Metric, symbol Device:R_US
- removed R19: 6.04kΩ, Resistor_SMD:R_0402_1005Metric, symbol Device:R_US
- removed R20, R21, R22, R23: 10Ω, Resistor_SMD:R_0402_1005Metric, symbol Device:R_US
- removed R31: 100kΩ, Resistor_SMD:R_0402_1005Metric, symbol Device:R_US
- removed R32, R33, R34, R35, R36, R37: 3.3kΩ, Resistor_SMD:R_0402_1005Metric, symbol Device:R_US
- removed R38: 330Ω, Resistor_SMD:R_0402_1005Metric, symbol Device:R_US
- removed TP1, TP12, TP17, TP2, TP21, TP23, TP24, TP25, TP26, TP27, TP28, TP29, TP3, TP30, TP31, TP32, TP33, TP34, TP35, TP36, TP37, TP38, TP39, TP4, TP40, TP5, TP6, TP8: TestPoint_Small, TestPoint:TestPoint_Pad_D1.0mm, symbol Connector:TestPoint_Small
- removed TP10, TP11, TP13, TP14, TP15, TP16, TP18, TP19, TP20, TP22, TP9: TestPoint, TestPoint:TestPoint_Pad_D3.0mm, symbol Connector:TestPoint
- removed U10: BQ76905RGRR, Library:VQFN20_RGR_TEX, symbol BMS:BQ76905RGRR
- removed U11: BQ25798RQMR, Library:RQM0029A-MFG, symbol BMS:BQ25798RQMR
- removed U14: TPS25730DREFR, Library:REF0038A-MFG, symbol BMS:TPS25730DREFR
- added TP6: TestPoint, TestPoint:TestPoint_Pad_D3.0mm, symbol Connector:TestPoint
- added TP8: TestPoint, TestPoint:TestPoint_THTPad_D3.0mm_Drill1.5mm, symbol Connector:TestPoint
- TP7: footprint TestPoint:TestPoint_Pad_D3.0mm -> TestPoint:TestPoint_THTPad_D3.0mm_Drill1.5mm
Connections:
- net PPHV is gone; now on net BAT+: TP7.1
- net VBUS: now also TP6.1
- new net BAT-: TP8.1
- no-connect marks 3 -> 1
Other:
- sheet Bucks renamed 5V Buck
- added sheet 3.3V Buck (3.3VBuck.kicad_sch)
- added sheet Charger (Bat_Charge.kicad_sch)
- added sheet PD Controller (PD.kicad_sch)
- added sheet Protector (Bat_Prot.kicad_sch)
- sheet 5V Buck ports: added 4.5V-28V IN, 5V OUT; removed PWR IN
