File: PCB/PiPortable.kicad_sch (KiCad schematic)
At the start: 4 parts, among them J11 USB_C_Receptacle_USB2.0

Commit message: Updated PCB
Parts:
- removed C18, C9: 100n, Capacitor_SMD:C_0402_1005Metric, symbol Device:C
- removed R9: 2.2K 1%, Resistor_SMD:R_0402_1005Metric, symbol Device:R
- added J23, J24: Conn_01x04_Pin, Connector_PinHeader_1.27mm:PinHeader_1x04_P1.27mm_Vertical, symbol Connector:Conn_01x04_Pin
- renumbered J11 to J1
Connections:
- net +5v renamed Power/VBUS
- net CC1 renamed Power/CC1
- net CC2 renamed Power/CC2
- net USB2_N renamed CM5_HighSpeed/USB2_N
- net USB2_P renamed CM5_HighSpeed/USB2_P
- new net IO Ports/H12: J23.1 (Pin_1)
- new net IO Ports/H13: J23.2 (Pin_2)
- new net IO Ports/H14: J23.3 (Pin_3)
- new net IO Ports/H15: J23.4 (Pin_4)
- new net IO Ports/L12: J24.1 (Pin_1)
- new net IO Ports/L13: J24.2 (Pin_2)
- new net IO Ports/L14: J24.3 (Pin_3)
- new net IO Ports/L15: J24.4 (Pin_4)
- no-connect marks 2 -> 8
Other:
- sheet CM5_GPIO ( Ethernet, GPIO, SDCARD) ports: added CLK0, GPIO22, GPIO23, GPIO24, GPIO25, GPIOSCL, GPIOSDA, ID_SCL, ID_SDA, MISO0, MOSI0; removed +3.3v, +5v, CC1, CC2, GPIO_VREF, ID_SC, ID_SD
- sheet CM5_HighSpeed ports: added ID_SCL, ID_SDA, USB3D_N, USB3D_P, USB3RX_N, USB3RX_P, USB3TX_N, USB3TX_P; removed +3.3v, +5v, GPIO_VREF, ID_SC, ID_SD, PCIE_PWR_EN
- sheet IO Ports ports: added CLK, CS1, CS2, CS3, CS4, D+, D-, H12, H13, H14, H15, L12, L13, L14, L15, MISO, MOSI, SCL, SDA; removed none
- sheet PCIe-M2 ports: added none; removed +5v, PCIE_PWR_EN
- sheet Power ports: added CC1, CC2, D+, D-, SCL, SDA, VBUS; removed none
- note removed: "Discharge Resistor Needed by some Type C PSUs"
