File: PCB/USB Hub.kicad_sch (KiCad schematic)
At the start: 3 parts, among them U16 USB2514B_Bi, Y1 ABM8-24.000MHZ-D1G-T

Commit message: Updated PCB
Parts:
- added TP1, TP23, TP24, TP5: TestPoint_Small, TestPoint:TestPoint_Pad_D1.0mm, symbol Connector:TestPoint_Small
- R8: renamed from R13; footprint (none) -> Resistor_SMD:R_0603_1608Metric_Pad0.98x0.95mm_HandSolder
- renumbered U16 to U7
Connections:
- net at U7.13 (OCS_N1): now also TP24.1
- net at U7.17 (OCS_N2): now also TP23.1
- net at U7.19 (OCS_N3): now also TP5.1
- net at U7.21 (OCS_N4): now also TP1.1
- no-connect marks 0 -> 3
